File: Swipe_Embedded/ModdedDumbpad/dumbpad.kicad_pcb (KiCad board)
At the start: 2 copper layers, 108 x 78.7 mm, 31 parts

Commit message: *Refactored functions and devices to prepare for swipe pad integration *Improved pcb design
Parts:
- added ?: , , F.Cu at (93.5, 80.5)
- added ?: , , F.Cu at (91.0, 75.5)
- added ?: , , F.Cu at (91.0, 78.0)
- added ?: , , F.Cu at (91.0, 70.5)
- added ?: , , F.Cu at (93.5, 78.0)
- added ?: , , F.Cu at (93.5, 75.5)
- added ?: , , F.Cu at (93.5, 83.0)
- added ?: , , F.Cu at (91.0, 80.5)
- added ?: , , F.Cu at (93.5, 73.0)
- added ?: , , F.Cu at (91.0, 73.0)
- moved ? 3.50 mm to (96.0, 70.4)
- moved ? 3.50 mm to (96.0, 78.0)
- moved ? 3.50 mm to (96.0, 80.5)
- moved ? 3.50 mm to (96.0, 72.9)
- moved ? 3.50 mm to (96.0, 75.5)
- moved ? 3.50 mm to (96.0, 83.1)
- moved ? 3.35 mm to (91.0, 83.0)
- moved ? 2.69 mm to (93.5, 70.5)
- renumbered S10 to S1, S9 to S10, S8 to S3, S3 to S8, S1 to S9
Connections:
- ? pad 8: /GPIO33 -> /GPIO26
- ? pad 7: /GPIO32 -> /GPIO25
- ? pad 6: /GPI35 -> /GPIO32
- EXT1 pad 5: /GPI34 -> /GPIO34
- S1 pad S2: /GPIO12 -> /GPIO13
- S10 pad S2: /GPIO27 -> /GPIO12
- S16 pad S2: /GPIO25 -> /GPIO15
- S3 pad S2: /GPIO26 -> /GPIO14
- S8 pad S2: /GPIO3 -> /GPIO34
- S9 pad S2: /GPIO1 -> /GPIO27
Routing:
- net /GPIO34: track 0.00 -> 114.5 mm
- net /GPIO13: track 0.00 -> 99.7 mm
- net /GPIO3: track 84.1 -> 0.00 mm
- net /GPIO14: track 0.00 -> 67.7 mm
- net /GPIO1: track 62.8 -> 0.00 mm
- net /GPIO33: track 44.8 -> 0.00 mm
- net /GPI34: track 28.5 -> 0.00 mm
- net /GPIO26: track 75.2 -> 49.8 mm
- net /GPIO12: track 107.0 -> 85.0 mm
- net /GPIO25: track 60.5 -> 44.4 mm
- net +3V3: track 7.61 -> 23.6 mm
- net /GPIO27: track 92.7 -> 106.7 mm
- net /GND: track 498.6 -> 487.4 mm
- net /GPIO15: track 0.00 -> 6.37 mm
- net /GPIO32: track 39.3 -> 36.5 mm
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Other:
- board text added: "3V3"
- board text added: "Battery 400mAh"
- board text added: "DAC1"
- board text added: "DAC2"
- board text added: "GND"
- board text added: "GPIO32"
- board text added: "GPIO35 /BAT"
- board text added: "GPIO36 /PWR"
- board text added: "GPIO39"
- board text added: "OLIMEX ESP32-DevKit-LiPo-Rev.D"
